File: KiCad/rc_v1/_autosave-rc_v1.kicad_sch (KiCad schematic)
At the start: 33 parts, among them SW1 OS102011MS2Qxxx, SW10 TS12-1212, SW3 TS12-66, SW4 TS12-66, SW5 TS12-66, SW6 TS12-66, SW7 TS12-66, SW8 TS12-66, SW9 TS12-1212, U1 SDTx39xx2W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

Commit message: Backup
Will replace buffer with level shifter
Parts:
- added U4: TXS0102DCT, Package_SO:SSOP-8_2.95x2.8mm_P0.65mm, symbol Logic_LevelTranslator:TXS0102DCT
Changed lines of the file:
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@@
+    )
+  )
+  (symbol (lib_id "Logic_LevelTranslator:TXS0102DCT") (at 113.03 182.88 0) (unit 1)
+    (in_bom yes) (on_board yes) (dnp no) (fields_autoplaced)
+    (property "Reference" "U4" (at 115.2241 195.58 0)
+      (effects (font (size 1.27 1.27)) (justify left))
+    )
+    (property "Value" "TXS0102DCT" (at 115.2241 198.12 0)
+      (effects (font (size 1.27 1.27)) (justify left))
+    )
+    (property "Footprint" "Package_SO:SSOP-8_2.95x2.8mm_P0.65mm" (at 113.03 196.85 0)
+      (effects (font (size 1.27 1.27)) hide)
+    )
+    (property "Datasheet" "http://www.ti.com/lit/gpn/txs0102" (at 113.03 183.388 0)
+      (effects (font (size 1.27 1.27)) hide)
+    )
+    (pin "1")
+    (pin "2")
+    (pin "3")
+    (pin "4")
+    (pin "5")
+    (pin "6")
+    (pin "7")
+    (pin "8")
+    (instances
+      (project "rc_v1"
+        (path "/fd6b2e2b-03ff-4e23-9683-4bcf908740ea"
+          (reference "U4") (unit 1)
+        )
+      )
     )
   )
